File: solar-battery-load/solar-battery-load.kicad_pcb (KiCad board)
At the start: 2 copper layers, 80 x 80 mm, 153 parts, among them J2 Conn_01x01, J3 Conn_01x01, J4 Conn_01x01, J5 Conn_01x01, J6 Conn_01x01, J7 Conn_01x01, J8 Conn_01x01, J9 Conn_01x02, U1 LM317_TO-252, U10 LM317_TO-252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

Commit message: WIP
Other:
- board text added: "${HASH}"
- board text added: "${TAG}"
Changed lines of the file:
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@@
+		)
+	)
+	(gr_text "${TAG}"
+		(at -28.1 -37.1 0)
+		(layer "F.SilkS")
+		(effects
+			(font
+				(size 1.5 1.5)
+				(thickness 0.3)
+				(bold yes)
+			)
+			(justify left bottom)
+		)
+	)
+	(gr_text "${HASH}"
+		(at 17.5 38.3 0)
+		(layer "F.SilkS")
+		(effects
+			(font
+				(size 1.5 1.5)
+				(thickness 0.3)
+				(bold yes)
+			)
+			(justify left bottom)
 		)
 	)
